Commit message: Fix Robotiq gripper integration for Gazebo simulation
- Enable sim_gazebo and include_ros2_control for proper simulation
- Add Gazebo material properties for correct gripper visualization
- Fix duplicate gripper loading in ur_arm.urdf.xacro
- Configure GripperActionController with correct controller type
- Remove spawner namespace for simplified action interface

Gripper now displays correctly with proper colors in Gazebo and
provides working action interface at /robotiq_gripper_controller/gripper_cmd
compatible with MoveIt control.

🤖 Generated with [Claude Code](https://claude.com/claude-code)

Co-Authored-By: Claude Sonnet 4.5 <noreply@anthropic.com>

File: components/arm/robotiq_gripper.urdf.xacro (robot description, xacro)
@@ -18,20 +18,43 @@
                 prefix=""
                 parent="neo_gripper_mount_link"
-                sim_gazebo="false"
-                include_ros2_control="false"
+                sim_gazebo="true"
+                include_ros2_control="true"
                 use_fake_hardware="false"
                 com_port="/dev/ttyUSB0">
                 <origin xyz="0 0 0" rpy="0 0 -${pi / 2}"/>
             </xacro:robotiq_gripper>
-            <!-- Provide a simple Gazebo ros2_control block for the gripper -->
-            <ros2_control name="robotiq_gripper" type="system">
-                <hardware>
-                    <plugin>gazebo_ros2_control/GazeboSystem</plugin>
-                </hardware>
-                <joint name="finger_joint">
-                    <command_interface name="position"/>
-                    <state_interface name="position"/>
-                    <state_interface name="velocity"/>
-                </joint>
-            </ros2_control>
+            <!-- Gazebo-specific material properties for gripper -->
+            <gazebo reference="robotiq_140_base_link">
+                <material>Gazebo/DarkGrey</material>
+            </gazebo>
+            <gazebo reference="left_outer_knuckle">
+                <material>Gazebo/Grey</material>
+            </gazebo>
+            <gazebo reference="left_outer_finger">
+                <material>Gazebo/Black</material>
+            </gazebo>
+            <gazebo reference="left_inner_knuckle">
+                <material>Gazebo/Black</material>
+            </gazebo>
+            <gazebo reference="left_inner_finger">
+                <material>Gazebo/Black</material>
+            </gazebo>
+            <gazebo reference="left_inner_finger_pad">
+                <material>Gazebo/FlatBlack</material>
+            </gazebo>
+            <gazebo reference="right_outer_knuckle">
+                <material>Gazebo/Grey</material>
+            </gazebo>
+            <gazebo reference="right_outer_finger">
+                <material>Gazebo/Black</material>
+            </gazebo>
+            <gazebo reference="right_inner_knuckle">
+                <material>Gazebo/Black</material>
+            </gazebo>
+            <gazebo reference="right_inner_finger">
+                <material>Gazebo/Black</material>
+            </gazebo>
+            <gazebo reference="right_inner_finger_pad">
+                <material>Gazebo/FlatBlack</material>
+            </gazebo>
 </robot>

File: components/arm/ur_arm.urdf.xacro (robot description, xacro)
@@ -57,9 +57,5 @@
             <xacro:property name="gripper_type_value" value="$(arg gripper_type)"/>
             <!-- Include robotiq gripper if use_gripper is true OR gripper_type is set to 2f_140/2f_85 -->
-            <xacro:if value="${gripper_requested}">
-                <xacro:include filename="$(find neo_simulation2)/components/arm/robotiq_gripper.urdf.xacro"/>
-            </xacro:if>
-            <!-- Also include if gripper_type is specified (for MoveIt compatibility) -->
-            <xacro:if value="${gripper_type_value == '2f_140' or gripper_type_value == '2f_85'}">
+            <xacro:if value="${gripper_requested or gripper_type_value == '2f_140' or gripper_type_value == '2f_85'}">
                 <xacro:include filename="$(find neo_simulation2)/components/arm/robotiq_gripper.urdf.xacro"/>
             </xacro:if>
